File: ECAD/MainBoard_LEDlightTensegrity.kicad_pcb (KiCad board)
At the start: 2 copper layers, 0 parts

Commit message: Finished Layout
Parts:
- added IC1: ARDUINO_PRO_MINI_5V, ArduinoProMini-5V, F.Cu at (43.2, 31.8)
- added K1: CONN_3, SIL-3, F.Cu at (24.1, 27.9)
- added K2: CONN_3, SIL-3, F.Cu at (24.1, 35.6)
- added K3: CONN_3, SIL-3, F.Cu at (97.8, 33.8)
- added P1: CONN_2, SIL-2, F.Cu at (47.0, 20.3)
- added P2: CONN_2, SIL-2, F.Cu at (24.1, 43.9)
- added R1: 1.33K, SM0603, B.Cu at (51.9, 36.6)
- added R2: 0, SM0603, F.Cu at (36.6, 21.3)
- added R3: 0, SM0603, F.Cu at (32.5, 21.3)
- added R4: 300, SM0603, F.Cu at (52.8, 42.2)
- added SW1: SPST, SIL-2, F.Cu at (41.4, 20.3)
- added U1: OKL-T6-W12, OKL-T6-W12, B.Cu at (41.4, 36.1)
- added U2: CJ1117-3.3, SOT223, B.Cu at (59.2, 30.7)
- added U3: REDBOTACCEL, RedBotAccel, F.Cu at (82.5, 24.9)
- added U4: NRF24L01_MODULE, nRF24L01_Module, B.Cu at (66.0, 37.1)
Routing:
- net +5V: track 0.00 -> 128.3 mm, vias 0 -> 1
- net /LED: track 0.00 -> 52.0 mm
- net /SDA: track 0.00 -> 47.5 mm
- net /SCL: track 0.00 -> 46.4 mm
- net /CSN: track 0.00 -> 23.9 mm
- net /MOSI: track 0.00 -> 22.8 mm
- net /SCK: track 0.00 -> 21.0 mm
- net VCC: track 0.00 -> 19.6 mm
- net N-0000025: track 0.00 -> 17.0 mm
- net /MISO: track 0.00 -> 16.7 mm
- net N-0000036: track 0.00 -> 12.9 mm
- net N-0000038: track 0.00 -> 12.1 mm
- net N-0000037: track 0.00 -> 12.0 mm
- net /CE: track 0.00 -> 9.62 mm
- net N-0000035: track 0.00 -> 8.43 mm
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- added copper zone on B.Cu, net GND
Other:
- board outline added: 85 x 30 mm
- net class Default: trace_width 0.254 -> 0.5; via_dia 0.889 -> 1.5; via_drill 0.635 -> 0.85
- net class Power added: clearance 0.254, trace_width 1.5, via_dia 0.889, via_drill 0.635
