File: ECAD/$MainBoard_LEDlightTensegrity.sch (KiCad schematic (older format))
At the start: 15 parts, among them IC1 ARDUINO_PRO_MINI_5V, K1 CONN_3, K2 CONN_3, K3 CONN_3, P1 CONN_2, SW1 SPST, U1 OKL-T6-W12, U2 CJ1117-3.3, U3 REDBOTACCEL, U4 NRF24L01_MODULE

Commit message: Finished Layout
Parts:
- gave numbers to parts that had none: 1
Changed lines of the file:
@@
 $EndComp
 $Comp
-L +5V #PWR01
+L +5V #PWR7
 U 1 1 5400E7EC
 P 5700 1800
-F 0 "#PWR01" H 5700 1890 20  0001 C CNN
+F 0 "#PWR7" H 5700 1890 20  0001 C CNN
 F 1 "+5V" H 5700 1890 30  0000 C CNN
 F 2 "" H 5700 1800 60  0000 C CNN
@@
 $EndComp
 $Comp
-L +5V #PWR02
+L +5V #PWR2
 U 1 1 5400E7FF
 P 2750 5050
-F 0 "#PWR02" H 2750 5140 20  0001 C CNN
+F 0 "#PWR2" H 2750 5140 20  0001 C CNN
 F 1 "+5V" H 2750 5140 30  0000 C CNN
 F 2 "" H 2750 5050 60  0000 C CNN
@@
 $EndComp
 $Comp
-L +5V #PWR03
+L +5V #PWR8
 U 1 1 5400E805
 P 7300 5350
-F 0 "#PWR03" H 7300 5440 20  0001 C CNN
+F 0 "#PWR8" H 7300 5440 20  0001 C CNN
 F 1 "+5V" H 7300 5440 30  0000 C CNN
 F 2 "" H 7300 5350 60  0000 C CNN
@@
 $EndComp
 $Comp
-L GND #PWR04
+L GND #PWR3
 U 1 1 5400E856
 P 3200 3100
-F 0 "#PWR04" H 3200 3100 30  0001 C CNN
+F 0 "#PWR3" H 3200 3100 30  0001 C CNN
 F 1 "GND" H 3200 3030 30  0001 C CNN
 F 2 "" H 3200 3100 60  0000 C CNN
@@
 $EndComp
 $Comp
-L GND #PWR05
+L GND #PWR10
 U 1 1 5400E863
 P 7500 2200
-F 0 "#PWR05" H 7500 2200 30  0001 C CNN
+F 0 "#PWR10" H 7500 2200 30  0001 C CNN
 F 1 "GND" H 7500 2130 30  0001 C CNN
 F 2 "" H 7500 2200 60  0000 C CNN
@@
 $EndComp
 $Comp
-L GND #PWR06
+L GND #PWR11
 U 1 1 5400E869
 P 8200 4800
-F 0 "#PWR06" H 8200 4800 30  0001 C CNN
+F 0 "#PWR11" H 8200 4800 30  0001 C CNN
 F 1 "GND" H 8200 4730 30  0001 C CNN
 F 2 "" H 8200 4800 60  0000 C CNN
@@
 $EndComp
 $Comp
-L GND #PWR07
+L GND #PWR9
 U 1 1 5400E86F
 P 7300 5650
-F 0 "#PWR07" H 7300 5650 30  0001 C CNN
+F 0 "#PWR9" H 7300 5650 30  0001 C CNN
 F 1 "GND" H 7300 5580 30  0001 C CNN
 F 2 "" H 7300 5650 60  0000 C CNN
@@
 	7500 2100 7500 2200
 $Comp
-L GND #PWR08
+L GND #PWR5
 U 1 1 5400F248
 P 4250 3100
-F 0 "#PWR08" H 4250 3100 30  0001 C CNN
+F 0 "#PWR5" H 4250 3100 30  0001 C CNN
 F 1 "GND" H 4250 3030 30  0001 C CNN
 F 2 "" H 4250 3100 60  0000 C CNN
@@
 LED
 $Comp
-L +5V #PWR09
+L +5V #PWR12
 U 1 1 5400F33B
 P 8750 2200
-F 0 "#PWR09" H 8750 2290 20  0001 C CNN
+F 0 "#PWR12" H 8750 2290 20  0001 C CNN
 F 1 "+5V" H 8750 2290 30  0000 C CNN
 F 2 "" H 8750 2200 60  0000 C CNN
@@
 $EndComp
 $Comp
-L GND #PWR010
+L GND #PWR13
 U 1 1 5400F37B
 P 8750 2550
-F 0 "#PWR010" H 8750 2550 30  0001 C CNN
+F 0 "#PWR13" H 8750 2550 30  0001 C CNN
 F 1 "GND" H 8750 2480 30  0001 C CNN
 F 2 "" H 8750 2550 60  0000 C CNN
@@
 	3450 2050 3250 2050
 $Comp
-L GND #PWR011
+L GND #PWR1
 U 1 1 5400F65B
 P 2250 2400
-F 0 "#PWR011" H 2250 2400 30  0001 C CNN
+F 0 "#PWR1" H 2250 2400 30  0001 C CNN
 F 1 "GND" H 2250 2330 30  0001 C CNN
 F 2 "" H 2250 2400 60  0000 C CNN
@@
 NoConn ~ 9250 4200
 $Comp
-L VCC #PWR012
+L VCC #PWR6
 U 1 1 5400F962
 P 4400 1350
-F 0 "#PWR012" H 4400 1450 30  0001 C CNN
+F 0 "#PWR6" H 4400 1450 30  0001 C CNN
 F 1 "VCC" H 4400 1450 30  0000 C CNN
 F 2 "" H 4400 1350 60  0000 C CNN
@@
 	8800 5450 9100 5450
 $Comp
-L GND #PWR013
+L GND #PWR4
 U 1 1 5400FBB4
 P 3950 5400
-F 0 "#PWR013" H 3950 5400 30  0001 C CNN
+F 0 "#PWR4" H 3950 5400 30  0001 C CNN
 F 1 "GND" H 3950 5330 30  0001 C CNN
 F 2 "" H 3950 5400 60  0000 C CNN
@@
 	8200 1950 8200 3400
 $Comp
-L CONN_2 P?
+L CONN_2 P2
 U 1 1 54010B89
 P 8850 3050
-F 0 "P?" V 8800 3050 40  0000 C CNN
+F 0 "P2" V 8800 3050 40  0000 C CNN
 F 1 "CONN_2" V 8900 3050 40  0000 C CNN
 F 2 "" H 8850 3050 60  0000 C CNN
@@
 $EndComp
 $Comp
-L VCC #PWR?
+L VCC #PWR14
 U 1 1 54010B96
 P 9400 2850
-F 0 "#PWR?" H 9400 2950 30  0001 C CNN
+F 0 "#PWR14" H 9400 2950 30  0001 C CNN
 F 1 "VCC" H 9400 2950 30  0000 C CNN
 F 2 "" H 9400 2850 60  0000 C CNN
@@
 $EndComp
 $Comp
-L GND #PWR?
+L GND #PWR15
 U 1 1 54010B9C
 P 9400 3250
-F 0 "#PWR?" H 9400 3250 30  0001 C CNN
+F 0 "#PWR15" H 9400 3250 30  0001 C CNN
 F 1 "GND" H 9400 3180 30  0001 C CNN
 F 2 "" H 9400 3250 60  0000 C CNN

Commit message: Added Protection Diode and Secondary Battery Path
Added Reverse Voltage Protection Diode. Also added second battery input
if only two batteries are used vs 4 total (2x on each side). Added
footprint for diode DO-214AB
Parts:
- added D1: DIODE, ~, symbol DIODE
- added P3: CONN_2, symbol CONN_2
Connections:
- net GND: now also P3.1 (P1); no longer P2.1 (P1)
- net VCC: now also D1.1 (A); no longer U1.2 (VIN)
- new net: D1.2 (K), U1.2 (VIN)
- new net VAA: P2.1 (P1), P3.2 (PM)
Changed lines of the file:
@@
 Sheet 1 1
 Title ""
-Date "29 aug 2014"
+Date "31 aug 2014"
 Rev ""
 Comp ""
@@
 $EndComp
 $Comp
-L +5V #PWR7
+L +5V #PWR01
 U 1 1 5400E7EC
 P 5700 1800
-F 0 "#PWR7" H 5700 1890 20  0001 C CNN
+F 0 "#PWR01" H 5700 1890 20  0001 C CNN
 F 1 "+5V" H 5700 1890 30  0000 C CNN
 F 2 "" H 5700 1800 60  0000 C CNN
@@
 $EndComp
 $Comp
-L +5V #PWR2
+L +5V #PWR02
 U 1 1 5400E7FF
 P 2750 5050
-F 0 "#PWR2" H 2750 5140 20  0001 C CNN
+F 0 "#PWR02" H 2750 5140 20  0001 C CNN
 F 1 "+5V" H 2750 5140 30  0000 C CNN
 F 2 "" H 2750 5050 60  0000 C CNN
@@
 $EndComp
 $Comp
-L +5V #PWR8
+L +5V #PWR03
 U 1 1 5400E805
 P 7300 5350
-F 0 "#PWR8" H 7300 5440 20  0001 C CNN
+F 0 "#PWR03" H 7300 5440 20  0001 C CNN
 F 1 "+5V" H 7300 5440 30  0000 C CNN
 F 2 "" H 7300 5350 60  0000 C CNN
@@
 $EndComp
 $Comp
-L GND #PWR3
+L GND #PWR04
 U 1 1 5400E856
 P 3200 3100
-F 0 "#PWR3" H 3200 3100 30  0001 C CNN
+F 0 "#PWR04" H 3200 3100 30  0001 C CNN
 F 1 "GND" H 3200 3030 30  0001 C CNN
 F 2 "" H 3200 3100 60  0000 C CNN
@@
 $EndComp
 $Comp
-L GND #PWR10
+L GND #PWR05
 U 1 1 5400E863
 P 7500 2200
-F 0 "#PWR10" H 7500 2200 30  0001 C CNN
+F 0 "#PWR05" H 7500 2200 30  0001 C CNN
 F 1 "GND" H 7500 2130 30  0001 C CNN
 F 2 "" H 7500 2200 60  0000 C CNN
@@
 $EndComp
 $Comp
-L GND #PWR11
+L GND #PWR06
 U 1 1 5400E869
 P 8200 4800
-F 0 "#PWR11" H 8200 4800 30  0001 C CNN
+F 0 "#PWR06" H 8200 4800 30  0001 C CNN
 F 1 "GND" H 8200 4730 30  0001 C CNN
 F 2 "" H 8200 4800 60  0000 C CNN
@@
 $EndComp
 $Comp
-L GND #PWR9
+L GND #PWR07
 U 1 1 5400E86F
 P 7300 5650
-F 0 "#PWR9" H 7300 5650 30  0001 C CNN
+F 0 "#PWR07" H 7300 5650 30  0001 C CNN
 F 1 "GND" H 7300 5580 30  0001 C CNN
 F 2 "" H 7300 5650 60  0000 C CNN
@@
 	7500 2100 7500 2200
 $Comp
-L GND #PWR5
+L GND #PWR08
 U 1 1 5400F248
 P 4250 3100
-F 0 "#PWR5" H 4250 3100 30  0001 C CNN
+F 0 "#PWR08" H 4250 3100 30  0001 C CNN
 F 1 "GND" H 4250 3030 30  0001 C CNN
 F 2 "" H 4250 3100 60  0000 C CNN
@@
 LED
 $Comp
-L +5V #PWR12
+L +5V #PWR09
 U 1 1 5400F33B
 P 8750 2200
-F 0 "#PWR12" H 8750 2290 20  0001 C CNN
+F 0 "#PWR09" H 8750 2290 20  0001 C CNN
 F 1 "+5V" H 8750 2290 30  0000 C CNN
 F 2 "" H 8750 2200 60  0000 C CNN
@@
 $EndComp
 $Comp
-L GND #PWR13
+L GND #PWR010
 U 1 1 5400F37B
 P 8750 2550
-F 0 "#PWR13" H 8750 2550 30  0001 C CNN
+F 0 "#PWR010" H 8750 2550 30  0001 C CNN
 F 1 "GND" H 8750 2480 30  0001 C CNN
 F 2 "" H 8750 2550 60  0000 C CNN
@@
 	3450 2050 3250 2050
 $Comp
-L GND #PWR1
+L GND #PWR011
 U 1 1 5400F65B
 P 2250 2400
-F 0 "#PWR1" H 2250 2400 30  0001 C CNN
+F 0 "#PWR011" H 2250 2400 30  0001 C CNN
 F 1 "GND" H 2250 2330 30  0001 C CNN
 F 2 "" H 2250 2400 60  0000 C CNN
@@
 	5800 2250 5800 2450
 NoConn ~ 9250 4200
-$Comp
-L VCC #PWR6
-U 1 1 5400F962
-P 4400 1350
-F 0 "#PWR6" H 4400 1450 30  0001 C CNN
-F 1 "VCC" H 4400 1450 30  0000 C CNN
-F 2 "" H 4400 1350 60  0000 C CNN
-F 3 "" H 4400 1350 60  0000 C CNN
-	1    4400 1350
-	1    0    0    -1
-$EndComp
-Wire Wire Line
-	4400 1350 4400 1500
 Wire Wire Line
 	3850 4700 4200 4700
@@
 	8800 5450 9100 5450
 $Comp
-L GND #PWR4
+L GND #PWR012
 U 1 1 5400FBB4
 P 3950 5400
-F 0 "#PWR4" H 3950 5400 30  0001 C CNN
+F 0 "#PWR012" H 3950 5400 30  0001 C CNN
 F 1 "GND" H 3950 5330 30  0001 C CNN
 F 2 "" H 3950 5400 60  0000 C CNN
@@
 $EndComp
 $Comp
-L VCC #PWR14
+L VCC #PWR013
 U 1 1 54010B96
 P 9400 2850
-F 0 "#PWR14" H 9400 2950 30  0001 C CNN
+F 0 "#PWR013" H 9400 2950 30  0001 C CNN
 F 1 "VCC" H 9400 2950 30  0000 C CNN
 F 2 "" H 9400 2850 60  0000 C CNN
@@
 $EndComp
 $Comp
-L GND #PWR15
+L GND #PWR014
 U 1 1 54010B9C
+P 10250 3250
+F 0 "#PWR014" H 10250 3250 30  0001 C CNN
+F 1 "GND" H 10250 3180 30  0001 C CNN
+F 2 "" H 10250 3250 60  0000 C CNN
+F 3 "" H 10250 3250 60  0000 C CNN
+	1    10250 3250
+	1    0    0    -1
+$EndComp
+Wire Wire Line
+	9400 2850 9400 2950
+Wire Wire Line
+	9400 2950 9200 2950
+$Comp
+L DIODE D1
+U 1 1 54026191
+P 4400 1200
+F 0 "D1" H 4400 1300 40  0000 C CNN
+F 1 "DIODE" H 4400 1100 40  0000 C CNN
+F 2 "~" H 4400 1200 60  0000 C CNN
+F 3 "~" H 4400 1200 60  0000 C CNN
+	1    4400 1200
+	0    1    1    0
+$EndComp
+Wire Wire Line
+	4400 950  4400 1000
+Wire Wire Line
+	4400 1400 4400 1500
+$Comp
+L VCC #PWR015
+U 1 1 54026D5F
+P 4400 950
+F 0 "#PWR015" H 4400 1050 30  0001 C CNN
+F 1 "VCC" H 4400 1050 30  0000 C CNN
+F 2 "" H 4400 950 60  0000 C CNN
+F 3 "" H 4400 950 60  0000 C CNN
+	1    4400 950
+	1    0    0    -1
+$EndComp
+$Comp
+L VAA #PWR016
+U 1 1 54026D6E
 P 9400 3250
-F 0 "#PWR15" H 9400 3250 30  0001 C CNN
-F 1 "GND" H 9400 3180 30  0001 C CNN
+F 0 "#PWR016" H 9400 3310 30  0001 C CNN
+F 1 "VAA" H 9400 3360 30  0000 C CNN
 F 2 "" H 9400 3250 60  0000 C CNN
 F 3 "" H 9400 3250 60  0000 C CNN
 	1    9400 3250
-	1    0    0    -1
-$EndComp
-Wire Wire Line
-	9400 2850 9400 2950
-Wire Wire Line
-	9400 2950 9200 2950
+	-1   0    0    1
+$EndComp
+$Comp
+L VAA #PWR017
+U 1 1 54026DA9
+P 10250 2850
+F 0 "#PWR017" H 10250 2910 30  0001 C CNN
+F 1 "VAA" H 10250 2960 30  0000 C CNN
+F 2 "" H 10250 2850 60  0000 C CNN
+F 3 "" H 10250 2850 60  0000 C CNN
+	1    10250 2850
+	1    0    0    -1
+$EndComp
+$Comp
+L CONN_2 P3
+U 1 1 54026DAF
+P 9800 3050
+F 0 "P3" V 9750 3050 40  0000 C CNN
+F 1 "CONN_2" V 9850 3050 40  0000 C CNN
+F 2 "" H 9800 3050 60  0000 C CNN
+F 3 "" H 9800 3050 60  0000 C CNN
+	1    9800 3050
+	-1   0    0    1
+$EndComp
+Wire Wire Line
+	10250 2850 10250 2950
+Wire Wire Line
+	10250 2950 10150 2950
 Wire Wire Line
 	9200 3150 9400 3150
 Wire Wire Line
 	9400 3150 9400 3250
+Wire Wire Line
+	10150 3150 10250 3150
+Wire Wire Line
+	10250 3150 10250 3250
 $EndSCHEMATC
