File: ECAD/MainBoard_LEDlightTensegrity.sch (KiCad schematic (older format))
At the start: 15 parts, among them IC1 ARDUINO_PRO_MINI_5V, K1 CONN_3, K2 CONN_3, K3 CONN_3, P1 CONN_2, SW1 SPST, U1 OKL-T6-W12, U2 CJ1117-3.3, U3 REDBOTACCEL, U4 NRF24L01_MODULE

Commit message: Added Protection Diode and Secondary Battery Path
Added Reverse Voltage Protection Diode. Also added second battery input
if only two batteries are used vs 4 total (2x on each side). Added
footprint for diode DO-214AB
Parts:
- added D1: DIODE, ~, symbol DIODE
- added P?: CONN_2, symbol CONN_2
- gave numbers to parts that had none: 1
Connections:
- net GND: now also P?.1 (P1); no longer P2.1 (P1)
- net VCC: now also D1.1 (A); no longer U1.2 (VIN)
- new net: D1.2 (K), U1.2 (VIN)
- new net VAA: P2.1 (P1), P?.2 (PM)
Changed lines of the file:
@@
 Sheet 1 1
 Title ""
-Date "29 aug 2014"
+Date "31 aug 2014"
 Rev ""
 Comp ""
@@
 	5800 2250 5800 2450
 NoConn ~ 9250 4200
-$Comp
-L VCC #PWR012
-U 1 1 5400F962
-P 4400 1350
-F 0 "#PWR012" H 4400 1450 30  0001 C CNN
-F 1 "VCC" H 4400 1450 30  0000 C CNN
-F 2 "" H 4400 1350 60  0000 C CNN
-F 3 "" H 4400 1350 60  0000 C CNN
-	1    4400 1350
-	1    0    0    -1
-$EndComp
-Wire Wire Line
-	4400 1350 4400 1500
 Wire Wire Line
 	3850 4700 4200 4700
@@
 	8200 1950 8200 3400
 $Comp
-L CONN_2 P?
+L CONN_2 P2
 U 1 1 54010B89
 P 8850 3050
-F 0 "P?" V 8800 3050 40  0000 C CNN
+F 0 "P2" V 8800 3050 40  0000 C CNN
 F 1 "CONN_2" V 8900 3050 40  0000 C CNN
 F 2 "" H 8850 3050 60  0000 C CNN
@@
 $EndComp
 $Comp
-L VCC #PWR?
+L VCC #PWR014
 U 1 1 54010B96
 P 9400 2850
-F 0 "#PWR?" H 9400 2950 30  0001 C CNN
+F 0 "#PWR014" H 9400 2950 30  0001 C CNN
 F 1 "VCC" H 9400 2950 30  0000 C CNN
 F 2 "" H 9400 2850 60  0000 C CNN
@@
 $EndComp
 $Comp
-L GND #PWR?
+L GND #PWR015
 U 1 1 54010B9C
+P 10250 3250
+F 0 "#PWR015" H 10250 3250 30  0001 C CNN
+F 1 "GND" H 10250 3180 30  0001 C CNN
+F 2 "" H 10250 3250 60  0000 C CNN
+F 3 "" H 10250 3250 60  0000 C CNN
+	1    10250 3250
+	1    0    0    -1
+$EndComp
+Wire Wire Line
+	9400 2850 9400 2950
+Wire Wire Line
+	9400 2950 9200 2950
+$Comp
+L DIODE D1
+U 1 1 54026191
+P 4400 1200
+F 0 "D1" H 4400 1300 40  0000 C CNN
+F 1 "DIODE" H 4400 1100 40  0000 C CNN
+F 2 "~" H 4400 1200 60  0000 C CNN
+F 3 "~" H 4400 1200 60  0000 C CNN
+	1    4400 1200
+	0    1    1    0
+$EndComp
+Wire Wire Line
+	4400 950  4400 1000
+Wire Wire Line
+	4400 1400 4400 1500
+$Comp
+L VCC #PWR?
+U 1 1 54026D5F
+P 4400 950
+F 0 "#PWR?" H 4400 1050 30  0001 C CNN
+F 1 "VCC" H 4400 1050 30  0000 C CNN
+F 2 "" H 4400 950 60  0000 C CNN
+F 3 "" H 4400 950 60  0000 C CNN
+	1    4400 950
+	1    0    0    -1
+$EndComp
+$Comp
+L VAA #PWR?
+U 1 1 54026D6E
 P 9400 3250
-F 0 "#PWR?" H 9400 3250 30  0001 C CNN
-F 1 "GND" H 9400 3180 30  0001 C CNN
+F 0 "#PWR?" H 9400 3310 30  0001 C CNN
+F 1 "VAA" H 9400 3360 30  0000 C CNN
 F 2 "" H 9400 3250 60  0000 C CNN
 F 3 "" H 9400 3250 60  0000 C CNN
 	1    9400 3250
-	1    0    0    -1
-$EndComp
-Wire Wire Line
-	9400 2850 9400 2950
-Wire Wire Line
-	9400 2950 9200 2950
+	-1   0    0    1
+$EndComp
+$Comp
+L VAA #PWR?
+U 1 1 54026DA9
+P 10250 2850
+F 0 "#PWR?" H 10250 2910 30  0001 C CNN
+F 1 "VAA" H 10250 2960 30  0000 C CNN
+F 2 "" H 10250 2850 60  0000 C CNN
+F 3 "" H 10250 2850 60  0000 C CNN
+	1    10250 2850
+	1    0    0    -1
+$EndComp
+$Comp
+L CONN_2 P?
+U 1 1 54026DAF
+P 9800 3050
+F 0 "P?" V 9750 3050 40  0000 C CNN
+F 1 "CONN_2" V 9850 3050 40  0000 C CNN
+F 2 "" H 9800 3050 60  0000 C CNN
+F 3 "" H 9800 3050 60  0000 C CNN
+	1    9800 3050
+	-1   0    0    1
+$EndComp
+Wire Wire Line
+	10250 2850 10250 2950
+Wire Wire Line
+	10250 2950 10150 2950
 Wire Wire Line
 	9200 3150 9400 3150
 Wire Wire Line
 	9400 3150 9400 3250
+Wire Wire Line
+	10150 3150 10250 3150
+Wire Wire Line
+	10250 3150 10250 3250
 $EndSCHEMATC

Commit message: Added first push of Arduino control code
Simple Accelerometer + lights responding code to test tube segments
Parts:
- gave numbers to parts that had none: 1
Changed lines of the file:
@@
 	8800 5450 9100 5450
 $Comp
-L GND #PWR013
+L GND #PWR012
 U 1 1 5400FBB4
 P 3950 5400
-F 0 "#PWR013" H 3950 5400 30  0001 C CNN
+F 0 "#PWR012" H 3950 5400 30  0001 C CNN
 F 1 "GND" H 3950 5330 30  0001 C CNN
 F 2 "" H 3950 5400 60  0000 C CNN
@@
 $EndComp
 $Comp
-L VCC #PWR014
+L VCC #PWR013
 U 1 1 54010B96
 P 9400 2850
-F 0 "#PWR014" H 9400 2950 30  0001 C CNN
+F 0 "#PWR013" H 9400 2950 30  0001 C CNN
 F 1 "VCC" H 9400 2950 30  0000 C CNN
 F 2 "" H 9400 2850 60  0000 C CNN
@@
 $EndComp
 $Comp
-L GND #PWR015
+L GND #PWR014
 U 1 1 54010B9C
 P 10250 3250
-F 0 "#PWR015" H 10250 3250 30  0001 C CNN
+F 0 "#PWR014" H 10250 3250 30  0001 C CNN
 F 1 "GND" H 10250 3180 30  0001 C CNN
 F 2 "" H 10250 3250 60  0000 C CNN
@@
 	4400 1400 4400 1500
 $Comp
-L VCC #PWR?
+L VCC #PWR015
 U 1 1 54026D5F
 P 4400 950
-F 0 "#PWR?" H 4400 1050 30  0001 C CNN
+F 0 "#PWR015" H 4400 1050 30  0001 C CNN
 F 1 "VCC" H 4400 1050 30  0000 C CNN
 F 2 "" H 4400 950 60  0000 C CNN
@@
 $EndComp
 $Comp
-L VAA #PWR?
+L VAA #PWR016
 U 1 1 54026D6E
 P 9400 3250
-F 0 "#PWR?" H 9400 3310 30  0001 C CNN
+F 0 "#PWR016" H 9400 3310 30  0001 C CNN
 F 1 "VAA" H 9400 3360 30  0000 C CNN
 F 2 "" H 9400 3250 60  0000 C CNN
@@
 $EndComp
 $Comp
-L VAA #PWR?
+L VAA #PWR017
 U 1 1 54026DA9
 P 10250 2850
-F 0 "#PWR?" H 10250 2910 30  0001 C CNN
+F 0 "#PWR017" H 10250 2910 30  0001 C CNN
 F 1 "VAA" H 10250 2960 30  0000 C CNN
 F 2 "" H 10250 2850 60  0000 C CNN
@@
 $EndComp
 $Comp
-L CONN_2 P?
+L CONN_2 P3
 U 1 1 54026DAF
 P 9800 3050
-F 0 "P?" V 9750 3050 40  0000 C CNN
+F 0 "P3" V 9750 3050 40  0000 C CNN
 F 1 "CONN_2" V 9850 3050 40  0000 C CNN
 F 2 "" H 9800 3050 60  0000 C CNN
